File: switch.brd (EAGLE design)
At the start: 42.9 x 29.2 mm, 4 parts

Commit message: edited
Parts:
- added SL1: (no value), con-amp-quick:03P
Connections:
- new net N$2: SL1.2, X4.2
- new net N$5: SL1.3, U$1.P$6
- net N$4: now also SL1.1, U$1.P$7; no longer U$1.P$6, X4.2
Routing:
- net N$4: track 26.0 -> 7.62 mm
- net N$2: track 0.00 -> 18.4 mm
- net N$5: track 0.00 -> 10.2 mm
Changed lines of the file:
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@@
 <attribute name="OC_FARNELL" value="unknown" x="34.29" y="7.62" size="1.778" layer="27" rot="R270" display="off"/>
+</element>
+<element name="SL1" library="con-amp-quick" package="03P" value="" x="15.24" y="7.62" rot="R270">
+<attribute name="OC_NEWARK" value="unknown" x="15.24" y="7.62" size="1.778" layer="27" rot="R270" display="off"/>
+<attribute name="MPN" value="" x="15.24" y="7.62" size="1.778" layer="27" rot="R270" display="off"/>
+<attribute name="MF" value="" x="15.24" y="7.62" size="1.778" layer="27" rot="R270" display="off"/>
+<attribute name="OC_FARNELL" value="unknown" x="15.24" y="7.62" size="1.778" layer="27" rot="R270" display="off"/>
 </element>
 </elements>
@@
 <wire x1="21.59" y1="20.955" x2="21.59" y2="15.24" width="0.4064" layer="16"/>
 </signal>
+<signal name="N$2">
+<contactref element="X4" pad="2"/>
+<contactref element="SL1" pad="2"/>
+<wire x1="15.24" y1="7.62" x2="33.655" y2="7.62" width="0.4064" layer="16"/>
+</signal>
 <signal name="N$4">
+<contactref element="SL1" pad="1"/>
+<contactref element="U$1" pad="P$7"/>
+<wire x1="15.24" y1="10.16" x2="7.62" y2="10.16" width="0.4064" layer="16"/>
+</signal>
+<signal name="N$5">
+<contactref element="SL1" pad="3"/>
 <contactref element="U$1" pad="P$6"/>
-<contactref element="X4" pad="2"/>
-<wire x1="7.62" y1="7.62" x2="33.655" y2="7.62" width="0.4064" layer="16"/>
+<wire x1="7.62" y1="7.62" x2="11.43" y2="7.62" width="0.4064" layer="16"/>
+<wire x1="11.43" y1="7.62" x2="11.43" y2="5.08" width="0.4064" layer="16"/>
+<wire x1="11.43" y1="5.08" x2="15.24" y2="5.08" width="0.4064" layer="16"/>
 </signal>
 </signals>
