File: switch.sch (EAGLE design)
At the start: 4 parts

Commit message: edited
Parts:
- added SL1: (no value), con-amp-quick:M03S
Connections:
- new net N$2: SL1-2.S, X4-2.KL
- new net N$5: SL1-3.S, U$1.GPIO0
- net N$4: now also SL1-1.S, U$1.GPIO2; no longer U$1.GPIO0, X4-2.KL
Changed lines of the file:
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@@
 <part name="X2" library="con-wago-508" deviceset="W237-02P" device=""/>
 <part name="X4" library="con-wago-508" deviceset="W237-3E" device=""/>
+<part name="SL1" library="con-amp-quick" deviceset="M03S" device=""/>
 </parts>
 <sheets>
@@
 <instance part="X4" gate="-2" x="-27.94" y="48.26"/>
 <instance part="X4" gate="-3" x="-27.94" y="43.18"/>
+<instance part="SL1" gate="-1" x="2.54" y="66.04"/>
+<instance part="SL1" gate="-2" x="2.54" y="60.96"/>
+<instance part="SL1" gate="-3" x="2.54" y="55.88"/>
 </instances>
 <busses>
@@
 </segment>
 </net>
+<net name="N$2" class="0">
+<segment>
+<pinref part="X4" gate="-2" pin="KL"/>
+<wire x1="-22.86" y1="48.26" x2="10.16" y2="48.26" width="0.1524" layer="91"/>
+<wire x1="10.16" y1="48.26" x2="10.16" y2="60.96" width="0.1524" layer="91"/>
+<pinref part="SL1" gate="-2" pin="S"/>
+<wire x1="10.16" y1="60.96" x2="7.62" y2="60.96" width="0.1524" layer="91"/>
+</segment>
+</net>
 <net name="N$4" class="0">
 <segment>
-<pinref part="U$1" gate="G$1" pin="GPIO0"/>
-<wire x1="12.7" y1="48.26" x2="12.7" y2="60.96" width="0.1524" layer="91"/>
-<wire x1="-22.86" y1="48.26" x2="12.7" y2="48.26" width="0.1524" layer="91"/>
-<pinref part="X4" gate="-2" pin="KL"/>
+<pinref part="SL1" gate="-1" pin="S"/>
+<pinref part="U$1" gate="G$1" pin="GPIO2"/>
+<wire x1="7.62" y1="66.04" x2="12.7" y2="66.04" width="0.1524" layer="91"/>
 </segment>
 </net>
+<net name="N$5" class="0">
+<segment>
+<pinref part="SL1" gate="-3" pin="S"/>
+<pinref part="U$1" gate="G$1" pin="GPIO0"/>
+<wire x1="7.62" y1="55.88" x2="12.7" y2="55.88" width="0.1524" layer="91"/>
+<wire x1="12.7" y1="55.88" x2="12.7" y2="60.96" width="0.1524" layer="91"/>
+</segment>
+</net>
